Commit message: Merge the walking G1's fixed upper body into its pelvis
prepare_model.py now merges the 18 fixed-joint links on the pelvis, as the
upstream MJCF does, and checks the merged mass, centre of mass and inertia
against the MJCF's pelvis inertial. The articulation drops from 31 links to
13; walking is unchanged and a step costs about 40% less.

Co-Authored-By: Claude Opus 5.5 <noreply@anthropic.com>
Claude-Session: https://claude.ai/code/session_01ALg7o42ifcSeZyjfQywGwo

File: assets/robots/g1_description/g1_12dof.rne.urdf (robot description, URDF)
Before this commit: robot g1_12dof, 31 links, 30 joints
Links:
- removed link d435_link
- removed link head_link
- removed link imu_in_pelvis
- removed link imu_in_torso
- removed link left_elbow_link
- removed link left_shoulder_pitch_link
- removed link left_shoulder_roll_link
- removed link left_shoulder_yaw_link
- removed link left_wrist_roll_rubber_hand
- removed link logo_link
- removed link mid360_link
- removed link pelvis_contour_link
- removed link right_elbow_link
- removed link right_shoulder_pitch_link
- removed link right_shoulder_roll_link
- removed link right_shoulder_yaw_link
- removed link right_wrist_roll_rubber_hand
- removed link torso_link
- link pelvis: mass 3.813 -> 17.7348573; geometry collision cylinder length=0.03 radius=0.03; collision cylinder length=0.03 radius=0.03
Joints:
- removed joint d435_joint
- removed joint head_joint
- removed joint imu_in_pelvis_joint
- removed joint imu_in_torso_joint
- removed joint left_elbow_joint
- removed joint left_shoulder_pitch_joint
- removed joint left_shoulder_roll_joint
- removed joint left_shoulder_yaw_joint
- removed joint left_wrist_roll_joint
- removed joint logo_joint
- removed joint mid360_joint
- removed joint pelvis_contour_joint
- removed joint right_elbow_joint
- removed joint right_shoulder_pitch_joint
- removed joint right_shoulder_roll_joint
- removed joint right_shoulder_yaw_joint
- removed joint right_wrist_roll_joint
- removed joint waist_yaw_joint
